File: CircuitDiagrams/FINCH_Adapter_Board/FINCH_Adapter_Board.kicad_pcb (KiCad board)
At the start: 2 copper layers, 195 x 101.7 mm, 56 parts, among them J1 CONN_02X20, J2 CONN_02X25, J3 CONN_02X10, J4 CONN_01X07, J5 CONN_01X10, SW1 DIPS_04, U1 7417, U10 74LS163, U11 74LS163, U12 74LS163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

Commit message: todays work
Parts:
- C25, C26: footprint Capacitors_ThroughHole:C_Axial_D6_L11_P18 -> Discret:CP6
- moved C12 19.7 mm to (57.6, 68.9)
- moved C18 19.7 mm to (60.2, 107.0)
- moved C19 19.7 mm to (57.6, 56.2)
- moved C20 19.7 mm to (57.6, 43.5)
- moved C10 19.7 mm to (57.6, 94.3)
- moved C11 19.7 mm to (57.6, 81.6)
- moved U12 18.4 mm to (61.5, 74.0)
- moved U18 18.4 mm to (64.0, 112.1)
- moved U19 18.4 mm to (61.5, 61.3)
- moved U20 18.4 mm to (61.5, 48.6)
- moved U10 18.4 mm to (61.5, 99.4)
- moved U11 18.4 mm to (61.5, 86.9)
- moved C24 17.2 mm to (83.0, 107.0)
- moved C25 15.6 mm to (99.7, 63.8)
- moved C26 13.3 mm to (113.7, 58.7)
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Other:
- board text added: "+"

Commit message: todays work I
Parts:
- added REF**: eMountingHole_3.2mm_M3, Mounting_Holes:MountingHole_3.2mm_M3, F.Cu at (49.5, 52.6)
- added REF**: eMountingHole_3.2mm_M3, Mounting_Holes:MountingHole_3.2mm_M3, F.Cu at (49.5, 103.6)
- added REF**: eMountingHole_3.2mm_M3, Mounting_Holes:MountingHole_3.2mm_M3, F.Cu at (209.1, 103.6)
- J5: footprint Pin_Headers:Pin_Header_Straight_1x10 -> footprints:Conn_Molex-26-60-5100
- moved J5 14.0 mm to (94.9, 54.6)
- moved RN1 1.43 mm to (88.2, 56.1)
- moved C26 1.40 mm to (113.7, 60.1)
- moved C25 0.73 mm to (99.7, 64.6)
Routing:
- net GND: track 0.00 -> 480.1 mm
Other:
- net class 24V added: clearance 0.3, trace_width 2.8, via_dia 1.8, via_drill 0.9
- net class 5V added: clearance 0.3, trace_width 1.5, via_dia 1.8, via_drill 0.9
- net class Default: clearance 0.2 -> 0.3; trace_width 0.25 -> 0.5; via_dia 0.6 -> 1.8; via_drill 0.4 -> 0.9
- net class GND added: clearance 0.3, trace_width 1.5, via_dia 1.8, via_drill 0.9
- rule trace_clearance: 0.2 -> 0.3
- board text added: "1"

Commit message: todays work II
Parts:
- moved R1 0.26 mm to (149.0, 105.7)
- turned R2 to 270 degrees
Routing:
- net GND: track 480.1 -> 1086.2 mm
- net VCC: track 0.00 -> 351.4 mm, vias 0 -> 2
- net -5V: track 0.00 -> 90.2 mm
- net Net-(J4-Pad6): track 0.00 -> 81.6 mm, vias 0 -> 1
- net Net-(J4-Pad4): track 0.00 -> 80.0 mm, vias 0 -> 1

Commit message: todays work with bottom restriction
Parts:
- J3: footprint Pin_Headers:Pin_Header_Straight_2x10 -> footprints:Conn_AMP-1-87456-6
- SW1: footprint Pin_Headers:Pin_Header_Straight_2x04 -> Buttons_Switches_ThroughHole:SW_DIP_x4_Slide
- moved SW1 0.45 mm to (192.8, 103.1), turned to 0 degrees
Routing:
- net Net-(U19-Pad15): track 0.00 -> 366.7 mm, vias 0 -> 1
- net Net-(U10-Pad2): track 0.00 -> 356.3 mm, vias 0 -> 2
- net HIGH_3: track 0.00 -> 354.7 mm, vias 0 -> 9
- net HIGH_2: track 0.00 -> 318.4 mm, vias 0 -> 4
- net VCC: track 351.4 -> 664.7 mm, vias 2 -> 4
- net GND: track 1086.2 -> 1354.2 mm, vias 0 -> 2
- net Net-(U12-Pad15): track 0.00 -> 229.4 mm, vias 0 -> 2
- net -5V: track 90.2 -> 318.0 mm, vias 0 -> 7
- net Net-(U17-Pad9): track 0.00 -> 227.4 mm, vias 0 -> 1
- net Net-(U17-Pad4): track 0.00 -> 224.8 mm, vias 0 -> 2
- net Net-(U10-Pad1): track 0.00 -> 207.3 mm, vias 0 -> 5
- net /MASTER_RESET: track 0.00 -> 184.2 mm, vias 0 -> 3
- net /FINCH_Adapter_Board_02//CTRL_UNITACK1: track 0.00 -> 173.1 mm, vias 0 -> 2
- net /FINCH_Adapter_Board_02//CTRL_UNITACK0: track 0.00 -> 155.0 mm, vias 0 -> 2
- net Net-(RN1-Pad2): track 0.00 -> 150.4 mm, vias 0 -> 1
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Other:
- net class 24V: clearance 0.3 -> 0.2
- net class 5V: clearance 0.3 -> 0.2
- net class Default: clearance 0.3 -> 0.2
- net class GND: clearance 0.3 -> 0.2
- rule trace_clearance: 0.3 -> 0.2

Commit message: todays work
Parts:
- renumbered REF** to MOUNT1, REF** to MOUNT2, REF** to MOUNT3
Routing:
- net /FINCH_Adapter_Board_02//CTRL_BI-DATA: track 12.6 -> 140.5 mm
- net /FINCH_Adapter_Board_02/CTRL_CB5: track 0.00 -> 105.0 mm, vias 0 -> 1
- net /FINCH_Adapter_Board_02/CTRL_CB3: track 0.00 -> 104.1 mm, vias 0 -> 1
- net /FINCH_Adapter_Board_02/CTRL_CB6: track 0.00 -> 100.8 mm, vias 0 -> 1
- net /FINCH_Adapter_Board_02/CTRL_CB2: track 0.00 -> 86.3 mm, vias 0 -> 1
- net /FINCH_Adapter_Board_02/CTRL_BI-DATA: track 5.93 -> 90.6 mm
- net /FINCH_Adapter_Board_02//CTRL_WRITE-CLK: track 3.88 -> 81.3 mm
- net /FINCH_Adapter_Board_02/CTRL_CB4: track 0.00 -> 74.3 mm, vias 0 -> 1
- net /FINCH_Adapter_Board_02/CTRL_READ_ENABLE: track 19.6 -> 73.6 mm, vias 0 -> 1
- net DRIVE_SELECT: track 107.4 -> 155.8 mm
- net /FINCH_Adapter_Board_02/CTRL_WRITE_ENABLE: track 14.9 -> 53.2 mm, vias 0 -> 1
- net /FINCH_Adapter_Board_02//CTRL_WRITE_ENABLE: track 5.93 -> 43.8 mm, vias 0 -> 1
- net /FINCH_Adapter_Board_02//CTRL_READ-ENABLE: track 56.2 -> 93.5 mm
- net WRITE_ENABLE: track 0.00 -> 34.7 mm, vias 0 -> 1
- net /FINCH_Adapter_Board_02/CTRL_WRITE-CLK: track 3.88 -> 31.3 mm, vias 0 -> 1
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
Commit message: todays work
Routing:
- net /FINCH_Adapter_Board_02/CTRL_CB1: track 0.00 -> 194.2 mm, vias 0 -> 1
- net /FINCH_Adapter_Board_02/CTRL_CB0: track 0.00 -> 185.9 mm, vias 0 -> 1
- net /FINCH_Adapter_Board_02//CTRL_CWD0: track 0.00 -> 128.3 mm, vias 0 -> 1
- net /FINCH_Adapter_Board_02//CTRL_INDEX: track 0.00 -> 114.6 mm, vias 0 -> 3
- net Net-(U14-Pad4): track 0.00 -> 93.6 mm
- net /FINCH_Adapter_Board_02//CTRL_ATTN: track 0.00 -> 79.2 mm, vias 0 -> 1
- net Net-(U16-Pad4): track 0.00 -> 72.2 mm
- net /FINCH_Adapter_Board_02//CTRL_CWD1: track 0.00 -> 66.7 mm, vias 0 -> 1
- net DRV_DATA_BYTE_CLOCK: track 148.9 -> 208.5 mm
- net /FINCH_Adapter_Board_02/CTRL_CB2: track 86.3 -> 140.9 mm
- net /FINCH_Adapter_Board_02//CTRL_SECTOR: track 0.00 -> 44.6 mm, vias 0 -> 1
- net /FINCH_Adapter_Board_02/DRV_CMD_READ_ENABLE: track 61.4 -> 96.3 mm
- net GND: track 1374.9 -> 1340.8 mm
- net DRIVE_SELECT: track 155.8 -> 184.1 mm, vias 2 -> 3
- net /INDEX: track 0.00 -> 24.6 mm
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
Commit message: todays work
Routing:
- net Net-(U10-Pad1): track 199.9 -> 245.3 mm
- net /MASTER_RESET: track 171.8 -> 216.1 mm, vias 0 -> 1
- net /FINCH_Adapter_Board_02/CTRL_CB2: track 140.9 -> 99.2 mm
- net Net-(U5-Pad7): track 0.00 -> 28.9 mm, vias 0 -> 1
- net HIGH_3: track 375.1 -> 394.5 mm, vias 5 -> 6
- net /FINCH_Adapter_Board_02//CTRL_MASTER_RESET: track 131.6 -> 140.7 mm
- net /FINCH_Adapter_Board_02//CTRL_CWD1: track 66.7 -> 75.3 mm
- net DRIVE_SELECT: track 184.1 -> 189.1 mm
- net Net-(U10-Pad2): track 354.1 -> 357.7 mm
- net Net-(U17-Pad4): track 223.5 -> 220.0 mm
- net Net-(U17-Pad9): track 226.7 -> 223.2 mm
- net Net-(U15-Pad6): track 120.7 -> 123.8 mm
- net VCC: track 664.4 -> 661.9 mm
- net /FINCH_Adapter_Board_02/DRV_CMD_STEP: track 32.2 -> 34.6 mm, vias 1 -> 0
- net DRV_DATA_BYTE_CLOCK: track 208.5 -> 210.6 mm
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
Commit message: todays work - now everything is connected and DRC is successful
Routing:
- net GND: track 1340.8 -> 1452.1 mm
- net Net-(U10-Pad2): track 357.7 -> 423.6 mm, vias 1 -> 4
- net Net-(U2-Pad9): track 0.00 -> 33.5 mm, vias 0 -> 1
- net -5V: track 300.3 -> 313.3 mm
- net Net-(U10-Pad1): track 245.3 -> 248.8 mm
- net /MASTER_RESET: track 216.1 -> 219.6 mm
- net /FINCH_Adapter_Board_02/CTRL_SYSTEMCLK: track 96.7 -> 94.0 mm
- net Net-(RN1-Pad2): track 151.0 -> 148.5 mm
- net Net-(U5-Pad7): track 28.9 -> 30.5 mm
- net HIGH_3: track 394.5 -> 395.7 mm
- net Net-(U19-Pad15): track 369.3 -> 368.1 mm
- net Net-(U15-Pad9): track 30.1 -> 28.9 mm
- net Net-(U15-Pad2): track 95.0 -> 95.7 mm
- net /FINCH_Adapter_Board_02//CTRL_CWD0: track 128.3 -> 128.9 mm
