File: CircuitDiagrams/S8000_CPU/S8000_CPU_03.kicad_sch (KiCad schematic)
At the start: 15 parts, among them U25 74138, U26 74138, U27 7432, U35 7407, U4 7421, U48 74374, U49 74374, U50 74374, U54 7427, U8 7432, U9 7400

Commit message: Add Page 6 (SIO 2+3), 7 (CTC 2 + PIO)
Connections:
- net NMI_SWITCH_NC renamed P2_NMI_SWITCH_NC
- net NMI_SWITCH_NO renamed P2_NMI_SWITCH_NO
Changed lines of the file:
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@@
 		)
 	)
-	(global_label "NMI_SWITCH_NC"
+	(global_label "P2_NMI_SWITCH_NC"
 		(shape input)
 		(at 59.69 271.78 180)
@@
 		)
 		(property "Intersheetrefs" "${INTERSHEET_REFS}"
-			(at 41.9486 271.78 0)
+			(at 38.5015 271.78 0)
 			(hide yes)
 			(show_name no)
@@
 		)
 	)
-	(global_label "NMI_SWITCH_NO"
+	(global_label "P2_NMI_SWITCH_NO"
 		(shape input)
 		(at 59.69 237.49 180)
@@
 		)
 		(property "Intersheetrefs" "${INTERSHEET_REFS}"
-			(at 41.8881 237.49 0)
+			(at 38.441 237.49 0)
 			(hide yes)
 			(show_name no)
