File: CircuitDiagrams/S8000_CPU/S8000_CPU_05.kicad_sch (KiCad schematic)
At the start: 22 parts, among them U104 7404, U105 26LS30, U106 26LS32, U107 26LS32, U125 26LS32, U126 26LS30, U127 7404, U128 26LS30, U92 Z80 SIO/2, U93 Z80 SIO/2

Commit message: Add Page 6 (SIO 2+3)
Parts:
- C59, C60, C62, C88, C89, C90, C91, C94, C95, C96, C97: footprint (none) -> Capacitor_THT:CP_Radial_D6.3mm_P2.50mm
- C61: renamed from C51; footprint (none) -> Capacitor_THT:CP_Radial_D6.3mm_P2.50mm
- U104, U127: footprint (none) -> Package_DIP:DIP-14_W7.62mm
- U105, U106, U107, U126, U128: footprint (none) -> Package_DIP:DIP-16_W7.62mm
- U125: footprint (none) -> Capacitor_THT:CP_Radial_D7.5mm_P2.50mm
- U92: footprint (none) -> Package_DIP:DIP-40_W15.24mm; Comment (none) -> SIO 1
- U93: footprint (none) -> Package_DIP:DIP-40_W15.24mm; Comment (none) -> SIO 0
Other:
- moved on the sheet: U105E, U106E, U107E, U125E, U126E, U128E

Commit message: Add Page 6 (SIO 2+3), 7 (CTC 2 + PIO)
Connections:
- net TERMO_CTS0 renamed P2_SIO_CTS0
- net TERMO_CTS1 renamed P2_SIO_CTS1
- net TERMO_CTS2 renamed P2_SIO_CTS2
- net TERMO_CTS3 renamed P2_SIO_CTS3
- net TERMO_DSR0 renamed P2_SIO_DSR0
- net TERMO_DSR1 renamed P2_SIO_DSR1
- net TERMO_DSR2 renamed P2_SIO_DSR2
- net TERMO_DSR3 renamed P2_SIO_DSR3
- net TERMO_DTR0 renamed P2_SIO_DTR0
- net TERMO_DTR1 renamed P2_SIO_DTR1
- net TERMO_DTR2 renamed P2_SIO_DTR2
- net TERMO_DTR3 renamed P2_SIO_DTR3
- net TERMO_RTS0 renamed P2_SIO_RTS0
- net TERMO_RTS1 renamed P2_SIO_RTS1
- net TERMO_RTS2 renamed P2_SIO_RTS2
- net TERMO_RTS3 renamed P2_SIO_RTS3
- net TERMO_RXD0 renamed P2_SIO_RXD0
- net TERMO_RXD1 renamed P2_SIO_RXD1
- net TERMO_RXD2 renamed P2_SIO_RXD2
- net TERMO_RXD3 renamed P2_SIO_RXD3
- net TERMO_TXD0 renamed P2_SIO_TXD0
- net TERMO_TXD1 renamed P2_SIO_TXD1
- net TERMO_TXD2 renamed P2_SIO_TXD2
- net TERMO_TXD3 renamed P2_SIO_TXD3
- net TERMO_TXRTN0 renamed P2_SIO_TXRTN0
- net TERMO_TXRTN1 renamed P2_SIO_TXRTN1
- net TERMO_TXRTN2 renamed P2_SIO_TXRTN2
- net TERMO_TXRTN3 renamed P2_SIO_TXRTN3
Changed lines of the file:
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@@
 		)
 	)
-	(global_label "TERMO_CTS3"
+	(global_label "P2_SIO_CTS3"
 		(shape output)
 		(at 533.4 287.02 0)
@@
 		)
 	)
-	(global_label "TERMO_RXD2"
+	(global_label "P2_SIO_RXD2"
 		(shape output)
 		(at 533.4 233.68 0)
@@
 		)
 	)
-	(global_label "TERMO_RTS2"
+	(global_label "P2_SIO_RTS2"
 		(shape input)
 		(at 533.4 248.92 0)
@@
 		)
 	)
-	(global_label "TERMO_RTS0"
+	(global_label "P2_SIO_RTS0"
 		(shape input)
 		(at 533.4 86.36 0)
@@
 		)
 	)
-	(global_label "TERMO_DSR0"
+	(global_label "P2_SIO_DSR0"
 		(shape output)
 		(at 533.4 55.88 0)
@@
 		)
 	)
-	(global_label "TERMO_TXD2"
+	(global_label "P2_SIO_TXD2"
 		(shape input)
 		(at 533.4 256.54 0)
@@
 		)
 	)
-	(global_label "TERMO_TXD1"
+	(global_label "P2_SIO_TXD1"
 		(shape input)
 		(at 533.4 154.94 0)
@@
 		)
 	)
-	(global_label "TERMO_RTS3"
+	(global_label "P2_SIO_RTS3"
 		(shape input)
 		(at 533.4 309.88 0)
@@
 		)
 	)
-	(global_label "TERMO_DTR2"
+	(global_label "P2_SIO_DTR2"
 		(shape input)
 		(at 533.4 241.3 0)
@@
 		)
 	)
-	(global_label "TERMO_RTS1"
+	(global_label "P2_SIO_RTS1"
 		(shape input)
 		(at 533.4 147.32 0)
@@
 		)
 	)
-	(global_label "TERMO_DTR0"
+	(global_label "P2_SIO_DTR0"
 		(shape input)
 		(at 533.4 78.74 0)
@@
 		)
 	)
-	(global_label "TERMO_TXRTN2"
+	(global_label "P2_SIO_TXRTN2"
 		(shape input)
 		(at 533.4 264.16 0)
@@
 		)
 	)
-	(global_label "TERMO_TXD3"
+	(global_label "P2_SIO_TXD3"
 		(shape input)
 		(at 533.4 317.5 0)
@@
 		)
 	)
-	(global_label "TERMO_TXRTN0"
+	(global_label "P2_SIO_TXRTN0"
 		(shape input)
 		(at 533.4 101.6 0)
@@
 		)
 	)
-	(global_label "TERMO_CTS0"
+	(global_label "P2_SIO_CTS0"
 		(shape output)
 		(at 533.4 63.5 0)
@@
 		)
 	)
-	(global_label "TERMO_DTR1"
+	(global_label "P2_SIO_DTR1"
 		(shape input)
 		(at 533.4 139.7 0)
@@
 		)
 	)
-	(global_label "TERMO_RXD3"
+	(global_label "P2_SIO_RXD3"
 		(shape output)
 		(at 533.4 294.64 0)
@@
 		)
 	)
-	(global_label "TERMO_RXD1"
+	(global_label "P2_SIO_RXD1"
 		(shape output)
 		(at 533.4 132.08 0)
@@
 		)
 	)
-	(global_label "TERMO_TXD0"
+	(global_label "P2_SIO_TXD0"
 		(shape input)
 		(at 533.4 93.98 0)
@@
 		)
 	)
-	(global_label "TERMO_DTR3"
+	(global_label "P2_SIO_DTR3"
 		(shape input)
 		(at 533.4 302.26 0)
@@
 		)
 	)
-	(global_label "TERMO_DSR1"
+	(global_label "P2_SIO_DSR1"
 		(shape output)
 		(at 533.4 116.84 0)
@@
 		)
 	)
-	(global_label "TERMO_DSR3"
+	(global_label "P2_SIO_DSR3"
 		(shape output)
 		(at 533.4 279.4 0)
@@
 		)
 	)
-	(global_label "TERMO_TXRTN3"
+	(global_label "P2_SIO_TXRTN3"
 		(shape input)
 		(at 533.4 325.12 0)
@@
 		)
 	)
-	(global_label "TERMO_TXRTN1"
+	(global_label "P2_SIO_TXRTN1"
 		(shape input)
 		(at 533.4 162.56 0)
@@
 		)
 	)
-	(global_label "TERMO_DSR2"
+	(global_label "P2_SIO_DSR2"
 		(shape output)
 		(at 533.4 218.44 0)
@@
 		)
 	)
-	(global_label "TERMO_CTS2"
+	(global_label "P2_SIO_CTS2"
 		(shape output)
 		(at 533.4 226.06 0)
@@
 		)
 	)
-	(global_label "TERMO_CTS1"
+	(global_label "P2_SIO_CTS1"
 		(shape output)
 		(at 533.4 124.46 0)
@@
 		)
 	)
-	(global_label "TERMO_RXD0"
+	(global_label "P2_SIO_RXD0"
 		(shape output)
 		(at 533.4 71.12 0)

Commit message: Add Page 8 MMU (in progress)
Connections:
- net SIO 1 IEO: now reaches U92.7 (IEO)
Changed lines of the file:
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@@
 		)
 	)
+	(text "(Sh. 14)"
+		(exclude_from_sim no)
+		(at 553.72 339.09 0)
+		(effects
+			(font
+				(size 1.27 1.27)
+			)
+			(justify left)
+		)
+	)
 	(text "(Sh. 2)"
 		(exclude_from_sim no)
@@
 	(wire
 		(pts
+			(xy 236.22 289.56) (xy 223.52 289.56)
+		)
+		(stroke
+			(width 0)
+			(type default)
+		)
+	)
+	(wire
+		(pts
 			(xy 236.22 243.84) (xy 196.85 243.84)
 		)
@@
 	(wire
 		(pts
+			(xy 223.52 289.56) (xy 223.52 339.09)
+		)
+		(stroke
+			(width 0)
+			(type default)
+		)
+	)
+	(wire
+		(pts
 			(xy 450.85 118.11) (xy 438.15 118.11)
 		)
@@
 	(wire
 		(pts
+			(xy 223.52 339.09) (xy 533.4 339.09)
+		)
+		(stroke
+			(width 0)
+			(type default)
+		)
+	)
+	(wire
+		(pts
 			(xy 355.6 124.46) (xy 431.8 124.46)
 		)
@@
 			)
 		)
+	)
+	(global_label "SIO 1 IEO"
+		(shape output)
+		(at 533.4 339.09 0)
+		(fields_autoplaced yes)
+		(effects
+			(font
+				(size 1.27 1.27)
+			)
+			(justify left)
+		)
+		(property "Intersheetrefs" "${INTERSHEET_REFS}"
+			(at 545.759 339.09 0)
+			(hide yes)
+			(show_name no)
+			(do_not_autoplace no)
+			(effects
+				(font
+					(size 1.27 1.27)
+				)
+				(justify left)
+			)
+		)
