File: CircuitDiagrams/S8000_CPU/S8000_CPU_04.kicad_sch (KiCad schematic)
At the start: 8 parts, among them U14 74113, U32 7404, U33 7411, U41 7432, U43 Z80 CTC, U44 Z80 CTC, U81 7414

Commit message: Add Page 5 (SIO 0+1)
Changed lines of the file:
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@@
 	(text "(Sh. 7,14)"
 		(exclude_from_sim no)
-		(at 553.72 228.854 0)
+		(at 553.72 228.6 0)
 		(effects
 			(font
@@
 	(text "(Sh. 5)"
 		(exclude_from_sim no)
-		(at 553.72 218.694 0)
+		(at 553.72 218.44 0)
 		(effects
 			(font
@@
 	(text "(Sh. 13)"
 		(exclude_from_sim no)
-		(at 553.72 278.384 0)
-		(effects
-			(font
-				(size 1.27 1.27)
-			)
-			(justify left)
-		)
-	)
-	(text "(Sh. 5)"
-		(exclude_from_sim no)
-		(at 553.72 216.154 0)
+		(at 553.72 278.13 0)
+		(effects
+			(font
+				(size 1.27 1.27)
+			)
+			(justify left)
+		)
+	)
+	(text "(Sh. 5)"
+		(exclude_from_sim no)
+		(at 553.72 215.9 0)
 		(effects
 			(font
@@
 	(text "(Sh. 5)"
 		(exclude_from_sim no)
-		(at 553.72 112.014 0)
+		(at 553.72 111.76 0)
 		(effects
 			(font
@@
 	(text "(Sh. 3,10,11)"
 		(exclude_from_sim no)
-		(at 553.72 332.994 0)
+		(at 553.72 332.74 0)
 		(effects
 			(font
@@
 	(text "(Sh. 13)"
 		(exclude_from_sim no)
-		(at 553.72 288.544 0)
-		(effects
-			(font
-				(size 1.27 1.27)
-			)
-			(justify left)
-		)
-	)
-	(text "(Sh. 5)"
-		(exclude_from_sim no)
-		(at 553.72 221.234 0)
+		(at 553.72 288.29 0)
+		(effects
+			(font
+				(size 1.27 1.27)
+			)
+			(justify left)
+		)
+	)
+	(text "(Sh. 5)"
+		(exclude_from_sim no)
+		(at 553.72 220.98 0)
 		(effects
 			(font
@@
 	(text "(Sh. 5)"
 		(exclude_from_sim no)
-		(at 553.72 109.474 0)
+		(at 553.72 109.22 0)
 		(effects
 			(font
@@
 	(text "(Sh. 5)"
 		(exclude_from_sim no)
-		(at 553.72 114.554 0)
+		(at 553.72 114.3 0)
 		(effects
 			(font
@@
 	(text "(Sh. 14)"
 		(exclude_from_sim no)
-		(at 553.72 122.174 0)
-		(effects
-			(font
+		(at 553.72 121.92 0)
+		(effects
+			(font

Commit message: Add Page 6 (SIO 2+3), 7 (CTC 2 + PIO)
Connections:
- net +5V: now also U44.13 (IEI)
Changed lines of the file:
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@@
+	(symbol
+		(lib_id "power:+5V")
+		(at 236.22 121.92 90)
+		(unit 1)
+		(body_style 1)
+		(exclude_from_sim no)
+		(in_bom yes)
+		(on_board yes)
+		(in_pos_files yes)
+		(dnp no)
+		(fields_autoplaced yes)
+		(property "Reference" "#PWR06"
+			(at 240.03 121.92 0)
+			(hide yes)
+			(show_name no)
+			(do_not_autoplace no)
+			(effects
+				(font
+					(size 1.27 1.27)
+				)
+			)
+		)
+		(property "Value" "+5V"
+			(at 232.41 121.9199 90)
+			(show_name no)
+			(do_not_autoplace no)
+			(effects
+				(font
+					(size 1.27 1.27)
+				)
+				(justify left)
+			)
+		)
+		(property "Footprint" ""
+			(at 236.22 121.92 0)
+			(hide yes)
+			(show_name no)
+			(do_not_autoplace no)
+			(effects
+				(font
+					(size 1.27 1.27)
+				)
+			)
+		)
+		(property "Datasheet" ""
+			(at 236.22 121.92 0)
+			(hide yes)
+			(show_name no)
+			(do_not_autoplace no)
+			(effects
+				(font
+					(size 1.27 1.27)
+				)
+			)
+		)
+		(property "Description" "Power symbol creates a global label with name \"+5V\""
+			(at 236.22 121.92 0)
+			(hide yes)
+			(show_name no)
+			(do_not_autoplace no)
+			(effects
+				(font
+					(size 1.27 1.27)
+				)
+			)
+		)
+		(pin "1"
+		)
+		(instances
+			(project "S8000_CPU"
+				(path "/cee545ba-d57c-4b2c-bcb3-989a68b0ecfa/c84d5b69-34c9-4634-824a-223e6b3f03d4"
+					(reference "#PWR06")
+					(unit 1)
+				)
+			)
+		)
+	)
 	(symbol
 		(lib_id "power:+5V")

Commit message: Page 9 (EPROM + SRAM)
Other:
- note added: "(Sh. 9)"
Changed lines of the file:
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@@
 		)
 	)
-	(text "(Sh. 2)"
+	(text "(Sh. 9)"
 		(exclude_from_sim no)
 		(at 39.37 278.13 0)
