File: CircuitDiagrams/S8000_CPU/S8000_CPU_07.kicad_sch (KiCad schematic)
At the start: 17 parts, among them U1 Z80 PIO, U103 74244, U11 74240, U12 74240, U2 74LS244, U42 7408, U89 Z80 CTC

Commit message: Add Page 8 MMU (in progress)
Connections:
- net GND: now also U1.11 (GND)

Commit message: Footprints
Parts:
- E13, E14, E15, E16, E17, E18: footprint (none) -> Connector_PinHeader_2.54mm:PinHeader_1x01_P2.54mm_Horizontal
- U1: footprint (none) -> Package_DIP:DIP-40_W15.24mm
- U103, U11, U12: footprint (none) -> Package_DIP:DIP-20_W7.62mm
- U2: value 74LS244 -> 74244; footprint (none) -> Package_DIP:DIP-20_W7.62mm
- U42: footprint (none) -> Package_DIP:DIP-14_W7.62mm
Changed lines of the file:
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@@
 			)
 		)
-		(property "Footprint" ""
+		(property "Footprint" "Package_DIP:DIP-20_W7.62mm"
 			(at 411.48 203.2 0)
 			(hide yes)
@@
 			)
 		)
-		(property "Footprint" ""
+		(property "Footprint" "Package_DIP:DIP-20_W7.62mm"
 			(at 411.48 175.26 0)
 			(hide yes)
@@
 			)
 		)
-		(property "Footprint" ""
+		(property "Footprint" "Connector_PinHeader_2.54mm:PinHeader_1x01_P2.54mm_Horizontal"
 			(at 328.93 278.13 0)
 			(hide yes)
@@
 			)
 		)
-		(property "Footprint" ""
+		(property "Footprint" "Connector_PinHeader_2.54mm:PinHeader_1x01_P2.54mm_Horizontal"
 			(at 322.58 196.85 0)
 			(hide yes)
@@
 			)
 		)
-		(property "Footprint" ""
+		(property "Footprint" "Connector_PinHeader_2.54mm:PinHeader_1x01_P2.54mm_Horizontal"
 			(at 322.58 201.93 0)
 			(hide yes)
@@
 			)
 		)
-		(property "Footprint" ""
+		(property "Footprint" "Package_DIP:DIP-40_W15.24mm"
 			(at 256.54 241.3 0)
 			(hide yes)
@@
 			)
 		)
-		(property "Footprint" ""
+		(property "Footprint" "Package_DIP:DIP-14_W7.62mm"
 			(at 114.3 250.19 0)
 			(hide yes)
@@
 			)
 		)
-		(property "Footprint" ""
+		(property "Footprint" "Package_DIP:DIP-20_W7.62mm"
 			(at 358.14 213.36 0)
 			(hide yes)
@@
 			)
 		)
-		(property "Footprint" ""
+		(property "Footprint" "Package_DIP:DIP-20_W7.62mm"
 			(at 358.14 279.4 0)
 			(hide yes)
@@
 			)
 		)
-		(property "Footprint" ""
+		(property "Footprint" "Connector_PinHeader_2.54mm:PinHeader_1x01_P2.54mm_Horizontal"
 			(at 321.31 278.13 0)
 			(hide yes)
@@
 			)
 		)
-		(property "Footprint" ""
+		(property "Footprint" "Package_DIP:DIP-20_W7.62mm"
 			(at 384.81 284.48 0)
 			(hide yes)
@@
 			)
 		)
-		(property "Footprint" ""
+		(property "Footprint" "Connector_PinHeader_2.54mm:PinHeader_1x01_P2.54mm_Horizontal"
 			(at 330.2 196.85 0)
 			(hide yes)
@@
 			)
 		)
-		(property "Footprint" ""
+		(property "Footprint" "Connector_PinHeader_2.54mm:PinHeader_1x01_P2.54mm_Horizontal"
 			(at 328.93 283.21 0)
 			(hide yes)
@@
 			)
 		)
-		(property "Value" "74LS244"
+		(property "Value" "74244"
 			(at 413.6233 234.95 0)
 			(show_name no)
@@
 			)
 		)
-		(property "Footprint" ""
+		(property "Footprint" "Package_DIP:DIP-20_W7.62mm"
 			(at 411.48 252.73 0)
 			(hide yes)

Commit message: Page 10
Parts:
- removed U12: 74240, Package_DIP:DIP-20_W7.62mm, symbol 74xx:74LS240_Split
- added U12: 74244, symbol S8000:74LS244
- renumbered U2 to U108, U1 to U94
Connections:
- net E14_DEF: now also U12.9 (O0b)
- net GND: now also U12.19 (OEb)
- net P2_PIO_D.D./~{ACKNOWLEDGE}: now also U12.11 (I0b)
- no-connect marks 5 -> 11
Changed lines of the file:
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@@
 	(text "(Sh. 14)"
 		(exclude_from_sim no)
-		(at 553.72 306.07 0)
+		(at 553.72 309.88 0)
 		(effects
 			(font
@@
 	)
 	(junction
-		(at 201.93 231.14)
+		(at 455.93 284.48)
 		(diameter 0)
 		(color 0 0 0 0)
 	)
 	(junction
-		(at 483.87 199.39)
+		(at 201.93 231.14)
 		(diameter 0)
 		(color 0 0 0 0)
 	)
 	(junction
-		(at 455.93 284.48)
+		(at 483.87 199.39)
 		(diameter 0)
 		(color 0 0 0 0)
@@
 	)
 	(no_connect
+		(at 402.59 287.02)
+	)
+	(no_connect
+		(at 377.19 289.56)
+	)
+	(no_connect
+		(at 402.59 292.1)
+	)
+	(no_connect
+		(at 402.59 289.56)
+	)
+	(no_connect
+		(at 377.19 287.02)
+	)
+	(no_connect
 		(at 398.78 207.01)
 	)
@@
 	)
 	(no_connect
+		(at 377.19 292.1)
+	)
+	(no_connect
 		(at 276.86 233.68)
 	)
@@
 	(wire
 		(pts
+			(xy 402.59 284.48) (xy 455.93 284.48)
+		)
+		(stroke
+			(width 0)
+			(type default)
+		)
+	)
+	(wire
+		(pts
 			(xy 236.22 218.44) (xy 219.71 218.44)
 		)
@@
 	(wire
 		(pts
-			(xy 392.43 284.48) (xy 455.93 284.48)
-		)
-		(stroke
-			(width 0)
-			(type default)
-		)
-	)
-	(wire
-		(pts
 			(xy 382.27 173.99) (xy 398.78 173.99)
 		)
@@
 	(wire
 		(pts
-			(xy 227.33 306.07) (xy 533.4 306.07)
+			(xy 227.33 309.88) (xy 533.4 309.88)
 		)
 		(stroke
@@
 	(wire
 		(pts
-			(xy 227.33 279.4) (xy 227.33 306.07)
+			(xy 227.33 279.4) (xy 227.33 309.88)
 		)
 		(stroke
@@
 	(global_label "PIO 0 IEO"
 		(shape output)
-		(at 533.4 306.07 0)
+		(at 533.4 309.88 0)
 		(fields_autoplaced yes)
 		(effects
@@
 		)
 		(property "Intersheetrefs" "${INTERSHEET_REFS}"
-			(at 545.8195 306.07 0)
+			(at 545.8195 309.88 0)
 			(hide yes)
 			(show_name no)
@@
 		(dnp no)
 		(fields_autoplaced yes)
-		(property "Reference" "U1"
+		(property "Reference" "U94"
 			(at 258.6833 190.5 0)
 			(show_name no)
@@
 			(project "S8000_CPU"
 				(path "/cee545ba-d57c-4b2c-bcb3-989a68b0ecfa/0a5ad938-76de-4f46-b906-87758cba1508"
-					(reference "U1")
+					(reference "U94")
 					(unit 1)
 				)
@@
 	(symbol
 		(lib_id "power:GND")
-		(at 384.81 290.83 0)
-		(mirror y)
+		(at 389.89 300.99 0)
 		(unit 1)
 		(body_style 1)
@@
 		(fields_autoplaced yes)
 		(property "Reference" "#PWR015"
-			(at 384.81 297.18 0)
+			(at 389.89 307.34 0)
 			(hide yes)
 			(show_name no)
@@
 		)
 		(property "Value" "GND"
-			(at 384.81 295.91 0)
+			(at 389.89 306.07 0)
 			(show_name no)
 			(do_not_autoplace no)
@@
 		)
 		(property "Footprint" ""
-			(at 384.81 290.83 0)
+			(at 389.89 300.99 0)
 			(hide yes)
 			(show_name no)
@@
 		)
 		(property "Datasheet" ""
-			(at 384.81 290.83 0)
+			(at 389.89 300.99 0)
 			(hide yes)
 			(show_name no)
@@
 		)
 		(property "Description" "Power symbol creates a global label with name \"GND\" , ground"
-			(at 384.81 290.83 0)
+			(at 389.89 300.99 0)
 			(hide yes)
 			(show_name no)
@@
 	)
 	(symbol
+		(lib_id "S8000:74LS244")
+		(at 389.89 288.29 0)
+		(mirror y)
+		(unit 2)
+		(body_style 1)
+		(exclude_from_sim no)
+		(in_bom yes)
+		(on_board yes)
+		(in_pos_files yes)
+		(dnp no)
+		(fields_autoplaced yes)
+		(property "Reference" "U12"
+			(at 389.89 275.59 0)
+			(show_name no)
+			(do_not_autoplace no)
+			(effects
+				(font
+					(size 1.27 1.27)
+				)
+			)
+		)
+		(property "Value" "74244"
+			(at 389.89 278.13 0)
+			(show_name no)
+			(do_not_autoplace no)
+			(effects
+				(font
+					(size 1.27 1.27)
+				)
+			)
+		)
+		(property "Footprint" ""
+			(at 389.89 288.29 0)
+			(hide yes)
+			(show_name no)
+			(do_not_autoplace no)
+			(effects
+				(font
+					(size 1.27 1.27)
+				)
+			)
+		)
+		(property "Datasheet" ""
+			(at 389.89 288.29 0)
+			(hide yes)
+			(show_name no)
+			(do_not_autoplace no)
+			(effects
+				(font
+					(size 1.27 1.27)
+				)
+			)
+		)
+		(property "Description" ""
+			(at 389.89 288.29 0)
+			(hide yes)
+			(show_name no)
+			(do_not_autoplace no)
+			(effects
+				(font
+					(size 1.27 1.27)
+				)
+			)
+		)
+		(pin "3"
+		)
+		(pin "4"
+		)
+		(pin "17"
+		)
+		(pin "5"
+		)
+		(pin "13"
+		)
+		(pin "14"
+		)
+		(pin "11"
+		)
+		(pin "1"
+		)
+		(pin "10"
+		)
+		(pin "20"
+		)
+		(pin "18"
+		)
+		(pin "16"
+		)
+		(pin "6"
+		)
+		(pin "8"
+		)
+		(pin "2"
+		)
+		(pin "12"
+		)
+		(pin "19"
+		)
+		(pin "15"
+		)
+		(pin "9"
+		)
+		(pin "7"
+		)
+		(instances
+			(project "S8000_CPU"
+				(path "/cee545ba-d57c-4b2c-bcb3-989a68b0ecfa/0a5ad938-76de-4f46-b906-87758cba1508"
+					(reference "U12")
+					(unit 2)
+				)
+			)
+		)
+	)
+	(symbol
 		(lib_id "power:GND")
 		(at 256.54 134.62 0)
@@
 	)
 	(symbol
-		(lib_id "74xx:74LS240_Split")
-		(at 384.81 284.48 0)
-		(mirror y)
-		(unit 5)
-		(body_style 1)
-		(exclude_from_sim no)
-		(in_bom yes)
-		(on_board yes)
-		(in_pos_files yes)
-		(dnp no)
-		(fields_autoplaced yes)
-		(property "Reference" "U12"
-			(at 384.81 275.59 0)
-			(show_name no)
-			(do_not_autoplace no)
-			(effects
-				(font
-					(size 1.27 1.27)
-				)
-			)
-		)
-		(property "Value" "74240"
-			(at 384.81 278.13 0)
-			(show_name no)
-			(do_not_autoplace no)
-			(effects
-				(font
-					(size 1.27 1.27)
-				)
-			)
-		)
-		(property "Footprint" "Package_DIP:DIP-20_W7.62mm"
-			(at 384.81 284.48 0)
-			(hide yes)
-			(show_name no)
-			(do_not_autoplace no)
-			(effects
-				(font
-					(size 1.27 1.27)
-				)
-			)
-		)
-		(property "Datasheet" "http://www.ti.com/lit/ds/symlink/sn74ls240.pdf"
-			(at 384.81 284.48 0)
-			(hide yes)
-			(show_name no)
-			(do_not_autoplace no)
-			(effects
-				(font
-					(size 1.27 1.27)
-				)
-			)
-		)
-		(property "Description" "Octal Buffer and Line Driver With 3-State Output, active-low enables, inverting outputs, split symbol"
-			(at 384.81 284.48 0)
-			(hide yes)
-			(show_name no)
-			(do_not_autoplace no)
-			(effects
-				(font
-					(size 1.27 1.27)
-				)
-			)
-		)
-		(pin "16"
-		)
-		(pin "13"
-		)
-		(pin "7"
-		)
-		(pin "19"
-		)
-		(pin "10"
-		)
-		(pin "8"
-		)
-		(pin "14"
-		)
-		(pin "6"
-		)
-		(pin "3"
-		)
-		(pin "11"
-		)
-		(pin "9"
-		)
-		(pin "12"
-		)
-		(pin "2"
-		)
-		(pin "1"
-		)
-		(pin "18"
-		)
-		(pin "20"
-		)
-		(pin "4"
-		)
-		(pin "17"
-		)
-		(pin "15"
-		)
-		(pin "5"
-		)
-		(instances
-			(project "S8000_CPU"
-				(path "/cee545ba-d57c-4b2c-bcb3-989a68b0ecfa/0a5ad938-76de-4f46-b906-87758cba1508"
-					(reference "U12")
-					(unit 5)
-				)
-			)
-		)
-	)
-	(symbol
 		(lib_id "S8000:Terminal_Pin")
 		(at 330.2 196.85 0)
@@
 		(dnp no)
 		(fields_autoplaced yes)
-		(property "Reference" "U2"
+		(property "Reference" "U108"
 			(at 413.6233 232.41 0)
 			(show_name no)
@@
 			(project "S8000_CPU"
 				(path "/cee545ba-d57c-4b2c-bcb3-989a68b0ecfa/0a5ad938-76de-4f46-b906-87758cba1508"
-					(reference "U2")
+					(reference "U108")
 					(unit 1)
 				)
