File: CircuitDiagrams/S8000_CPU/S8000_CPU.kicad_sch (KiCad schematic)
At the start: 29 parts, among them U101 7404, U103 74244, U104 7404, U11 74240, U12 74240, U122 7404, U127 7404, U13 74113, U14 74113, U15 74113, U17 7400, U18 7402, U20 74113, U21 7432, U27 7432, U3 7408, U30 7410, U32 7404, U33 7411, U35 7407, U4 7421, U41 7432, U42 7408, U5 7408, U54 7427, U6 7402, U8 7432, U81 7414, U9 7400

Commit message: Page 9 (EPROM + SRAM)
Parts:
- added U56: 7432, symbol 74xx:74LS32
Connections:
- net +5V: now also U56.14 (VCC)
- net GND: now also U56.7 (GND)
Other:
- added sheet S8000 CPU 09 (S8000_CPU_09.kicad_sch)
- moved on the sheet: U54D
Changed lines of the file:
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@@
 	)
 	(junction
-		(at 177.8 152.4)
+		(at 171.45 152.4)
 		(diameter 0)
 		(color 0 0 0 0)
@@
 	)
 	(junction
-		(at 177.8 127)
+		(at 171.45 127)
 		(diameter 0)
 		(color 0 0 0 0)
@@
 	)
 	(junction
+		(at 182.88 152.4)
+		(diameter 0)
+		(color 0 0 0 0)
+	)
+	(junction
+		(at 182.88 127)
+		(diameter 0)
+		(color 0 0 0 0)
+	)
+	(junction
 		(at 218.44 111.76)
 		(diameter 0)
@@
 	(wire
 		(pts
-			(xy 148.59 152.4) (xy 223.52 152.4)
+			(xy 148.59 152.4) (xy 182.88 152.4)
 		)
 		(stroke
@@
 	(wire
 		(pts
+			(xy 182.88 127) (xy 223.52 127)
+		)
+		(stroke
+			(width 0)
+			(type default)
+		)
+	)
+	(wire
+		(pts
 			(xy 143.51 111.76) (xy 156.21 111.76)
 		)
@@
 	(wire
 		(pts
+			(xy 182.88 152.4) (xy 223.52 152.4)
+		)
+		(stroke
+			(width 0)
+			(type default)
+		)
+	)
+	(wire
+		(pts
 			(xy 241.3 86.36) (xy 252.73 86.36)
 		)
@@
 	(wire
 		(pts
-			(xy 148.59 127) (xy 223.52 127)
+			(xy 148.59 127) (xy 182.88 127)
 		)
 		(stroke
@@
 	(symbol
 		(lib_id "74xx:74LS27")
-		(at 177.8 139.7 0)
+		(at 171.45 139.7 0)
 		(unit 4)
 		(body_style 1)
@@
 		(dnp no)
 		(property "Reference" "U54"
-			(at 177.8 138.43 0)
+			(at 171.45 138.43 0)
 			(show_name no)
 			(do_not_autoplace no)
@@
 		)
 		(property "Value" "7427"
-			(at 177.8 140.97 0)
+			(at 171.45 140.97 0)
 			(show_name no)
 			(do_not_autoplace no)
@@
 		)
 		(property "Footprint" "Package_DIP:DIP-14_W7.62mm"
-			(at 177.8 139.7 0)
+			(at 171.45 139.7 0)
 			(hide yes)
 			(show_name no)
@@
 		)
 		(property "Datasheet" "http://www.ti.com/lit/gpn/sn74LS27"
-			(at 177.8 139.7 0)
+			(at 171.45 139.7 0)
 			(hide yes)
 			(show_name no)
@@
 		)
 		(property "Description" "Triple 3-input NOR"
-			(at 177.8 139.7 0)
+			(at 171.45 139.7 0)
 			(hide yes)
 			(show_name no)
@@
 	)
 	(symbol
+		(lib_id "74xx:74LS32")
+		(at 182.88 139.7 0)
+		(unit 5)
+		(body_style 1)
+		(exclude_from_sim no)
+		(in_bom yes)
+		(on_board yes)
+		(in_pos_files yes)
+		(dnp no)
+		(property "Reference" "U56"
+			(at 182.626 138.176 0)
+			(show_name no)
+			(do_not_autoplace no)
+			(effects
+				(font
+					(size 1.27 1.27)
+				)
+			)
+		)
+		(property "Value" "7432"
+			(at 182.626 140.716 0)
+			(show_name no)
+			(do_not_autoplace no)
+			(effects
+				(font
+					(size 1.27 1.27)
+				)
+			)
+		)
+		(property "Footprint" ""
+			(at 182.88 139.7 0)
+			(hide yes)
+			(show_name no)
+			(do_not_autoplace no)
+			(effects
+				(font
+					(size 1.27 1.27)
+				)
+			)
+		)
+		(property "Datasheet" "http://www.ti.com/lit/gpn/sn74LS32"
+			(at 182.88 139.7 0)
+			(hide yes)
+			(show_name no)
+			(do_not_autoplace no)
+			(effects
+				(font
+					(size 1.27 1.27)
+				)
+			)
+		)
+		(property "Description" "Quad 2-input OR"
+			(at 182.88 139.7 0)
+			(hide yes)
+			(show_name no)
+			(do_not_autoplace no)
+			(effects
+				(font
+					(size 1.27 1.27)
+				)
+			)
+		)
+		(pin "7"
+		)
+		(pin "12"
+		)
+		(pin "13"
+		)
+		(pin "11"
+		)
+		(pin "14"
+		)
+		(pin "2"
+		)
+		(pin "8"
+		)
+		(pin "5"
+		)
+		(pin "4"
+		)
+		(pin "3"
+		)
+		(pin "10"
+		)
+		(pin "1"
+		)
+		(pin "6"
+		)
+		(pin "9"
+		)
+		(instances
+			(project "S8000_CPU"
+				(path "/cee545ba-d57c-4b2c-bcb3-989a68b0ecfa"
+					(reference "U56")
+					(unit 5)
+				)
+			)
+		)
+	)
+	(symbol
 		(lib_id "74xx:74LS10")
 		(at 99.06 139.7 0)
@@
 				)
 			)
+		)
+	)
+	(sheet
+		(at 143.51 16.51)
+		(size 15.24 29.21)
+		(exclude_from_sim no)
+		(in_bom yes)
+		(on_board yes)
+		(dnp no)
+		(fields_autoplaced yes)
+		(stroke
+			(width 0.1524)
+			(type solid)
+		)
+		(fill
+			(color 0 0 0 0)
+		)
+		(property "Sheetname" "S8000 CPU 09"
+			(at 143.51 15.7984 0)
+			(show_name no)
+			(do_not_autoplace no)
+			(effects
+				(font
+					(size 1.27 1.27)
+				)
+				(justify left bottom)
+			)
+		)
+		(property "Sheetfile" "S8000_CPU_09.kicad_sch"
+			(at 143.51 46.3046 0)
+			(show_name no)
+			(do_not_autoplace no)
+			(effects
+				(font
+					(size 1.27 1.27)
+				)
+				(justify left top)
+			)
+		)
+		(instances
+			(project "S8000_CPU"
+				(path "/cee545ba-d57c-4b2c-bcb3-989a68b0ecfa"
+					(page "9")
+				)
+			)

Commit message: Page 10
Parts:
- removed U12: 74240, Package_DIP:DIP-20_W7.62mm, symbol 74xx:74LS240_Split
- removed U15: 74113, Package_DIP:DIP-14_W7.62mm, symbol 74xx:74LS113
- added U1, U29: 7404, symbol 74xx:74LS04
- added U12: 74244, symbol S8000:74LS244
- added U15: 7402, symbol 74xx:74LS02
- added U16: 7451, symbol 74xx:74LS51
- added U2, U23: 7410, symbol 74xx:74LS10
- added U22: 7432, symbol 74xx:74LS32
- added U34, U61: 74260, symbol S8000:74LS260
- added U38: 7408, symbol 74xx:74LS08
- added U7: 7474, symbol 74xx:74LS74
Connections:
- net +5V: now also U1.14 (VCC), U12.20 (VCC), U15.14 (VCC), U16.14 (VCC), U2.14 (VCC), U22.14 (VCC), U23.14 (VCC), U29.14 (VCC), U34.14 (VCC), U38.14 (VCC), U61.14 (VCC), U7.14 (VCC)
- net GND: now also U1.7 (GND), U12.10 (GND), U15.7 (GND), U16.7 (GND), U2.7 (GND), U22.7 (GND), U23.7 (GND), U29.7 (GND), U34.7 (GND), U38.7 (GND), U61.7 (GND), U7.7 (GND)
Other:
- added sheet S8000 CPU 10 (S8000_CPU_10.kicad_sch)
- moved on the sheet: U101G, U103C, U104G, U11I, U122G, U127G, U13C, U14C, U17E, U18E, U21E, U27E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

Commit message: Add page 1
Other:
- added sheet S8000 CPU 01 (S8000_CPU_01.kicad_sch)
Changed lines of the file:
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@@
+	)
+	(sheet
+		(at 92.71 63.5)
+		(size 12.7 13.97)
+		(exclude_from_sim no)
+		(in_bom yes)
+		(on_board yes)
+		(dnp no)
+		(fields_autoplaced yes)
+		(stroke
+			(width 0.1524)
+			(type solid)
+		)
+		(fill
+			(color 0 0 0 0)
+		)
+		(property "Sheetname" "S8000 CPU 01"
+			(at 92.71 62.7884 0)
+			(show_name no)
+			(do_not_autoplace no)
+			(effects
+				(font
+					(size 1.27 1.27)
+				)
+				(justify left bottom)
+			)
+		)
+		(property "Sheetfile" "S8000_CPU_01.kicad_sch"
+			(at 92.71 78.0546 0)
+			(hide yes)
+			(show_name no)
+			(do_not_autoplace no)
+			(effects
+				(font
+					(size 1.27 1.27)
+				)
+				(justify left top)
+			)
+		)
+		(instances
+			(project "S8000_CPU"
+				(path "/cee545ba-d57c-4b2c-bcb3-989a68b0ecfa"
+					(page "1")
+				)
+			)
+		)
 	)
 	(sheet
@@
 	(sheet_instances
 		(path "/"
-			(page "1")
-		)
-	)
+			(page "0")
+		)
+	)

Commit message: Add missing (still empty) pages
Other:
- added sheet S8000 CPU 11 (S8000_CPU_11.kicad_sch)
- added sheet S8000 CPU 12 (S8000_CPU_12.kicad_sch)
- added sheet S8000 CPU 13 (S8000_CPU_13.kicad_sch)
- added sheet S8000 CPU 14 (S8000_CPU_14.kicad_sch)

Commit message: page 11 done
Parts:
- added U78: 7411, symbol 74xx:74LS11
- added U83: 74113, symbol 74xx:74LS113
- added U95: 7404, symbol 74xx:74LS04
- added U96: 7408, symbol 74xx:74LS08
- added U97: 7474, symbol 74xx:74LS74
Connections:
- net +5V: now also U78.14 (VCC), U83.14 (VCC), U95.14 (VCC), U96.14 (VCC), U97.14 (VCC)
- net GND: now also U78.7 (GND), U83.7 (GND), U95.7 (GND), U96.7 (GND), U97.7 (GND)
Other:
- moved on the sheet: U101G, U103C, U104G, U122G, U127G, U81G

Commit message: page 12 done
Parts:
- removed U5: 7408, Package_DIP:DIP-14_W7.62mm, symbol 74xx:74LS08
- removed U6: 7402, Package_DIP:DIP-14_W7.62mm, symbol 74xx:74LS02
- removed U7: 7474, symbol 74xx:74LS74
- added U40, U5: 7474, symbol 74xx:74LS74
- added U45: 74133, symbol 74xx:74LS133
- added U6: 7400, symbol 74xx:74LS00
- added U7: 7420, symbol 74xx:74LS20
Connections:
- net +5V: now also U40.14 (VCC), U45.16 (VCC), U5.14 (VCC), U6.14 (VCC), U7.14 (VCC)
- net GND: now also U40.7 (GND), U45.8 (GND), U5.7 (GND), U6.7 (GND), U7.7 (GND)
Other:
- moved on the sheet: U38E, U41E
