File: CircuitDiagrams/S8000_CPU/S8000_CPU_02.kicad_sch (KiCad schematic)
At the start: 19 parts, among them U118 74244, U119 4.7k, U32 7404, U35 7407, U46 74245, U47 74373, U62 74373, U63 74245, U65 74374, U66 74374, U67 74244, U68 74240, U71 Z8001, U81 7414, U99 74241

Commit message: S8000 CPU schematics Page 3
Parts:
- renumbered TP4 to TP2, TP6 to TP3, TP7 to TP5

Commit message: Add Page 4
Connections:
- net ~{BD DATAEN} renamed ~{BD_DATAEN}
- net ~{INT} renamed PERIPH_~{VI}

Commit message: Add Page 5 (SIO 0+1)
Connections:
- net U119_PIN4: now reaches U119.4 (R3), U99.19 (OEb)
Other:
- note added: "PIN 19 FIXME check real board"
Changed lines of the file:
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@@
 		)
 	)
+	(text "PIN 19\nFIXME check\nreal board"
+		(exclude_from_sim no)
+		(at 188.976 195.072 0)
+		(effects
+			(font
+				(size 1.27 1.27)
+			)
+		)
+	)
 	(text ""
 		(exclude_from_sim no)
@@
 			)
 		)
+	)
+	(global_label "U119_PIN4"
+		(shape input)
+		(at 226.06 110.49 0)
+		(fields_autoplaced yes)
+		(effects
+			(font
+				(size 1.27 1.27)
+			)
+			(justify left)
+		)
+		(property "Intersheetrefs" "${INTERSHEET_REFS}"
+			(at 239.3866 110.49 0)
+			(hide yes)
+			(show_name no)
+			(do_not_autoplace no)
+			(effects
+				(font
+					(size 1.27 1.27)
+				)
+				(justify left)
+			)
+		)

Commit message: Page 10
Parts:
- renumbered U71 to U64

Commit message: page 11 done
Connections:
- net ~{MRESET}: now also U35.9; no longer U35.8
- net ~{RESET}: no longer U35.9
- new net ~{BUS_RESET}: U35.8
Changed lines of the file:
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@@
 	(text "(Sh. 4,5,6,7,8,11,14)"
 		(exclude_from_sim no)
-		(at 39.37 330.2 0)
+		(at 39.37 323.088 0)
 		(effects
 			(font
@@
 	(text "P1-1A"
 		(exclude_from_sim no)
-		(at 70.104 322.58 0)
+		(at 70.104 330.2 0)
 		(effects
 			(font
@@
 		)
 	)
-	(global_label "~{RESET}"
+	(global_label "~{MRESET}"
 		(shape input)
 		(at 207.01 322.58 180)
@@
 		)
 		(property "Intersheetrefs" "${INTERSHEET_REFS}"
-			(at 198.2797 322.58 0)
+			(at 196.8283 322.58 0)
 			(hide yes)
 			(show_name no)
@@
 	)
 	(global_label "BUS_~{WAIT}"
-		(shape output)
+		(shape input)
 		(at 59.69 289.56 180)
 		(fields_autoplaced yes)
@@
 		)
 	)
-	(global_label "~{RESET}"
+	(global_label "~{MRESET}"
 		(shape input)
 		(at 59.69 322.58 180)
@@
 		)
 		(property "Intersheetrefs" "${INTERSHEET_REFS}"
-			(at 50.9597 322.58 0)
+			(at 49.5083 322.58 0)
 			(hide yes)
 			(show_name no)
@@
 	)
 	(global_label "BUS_~{WAIT}"
-		(shape input)
+		(shape output)
 		(at 59.69 294.64 180)
 		(fields_autoplaced yes)
@@
 		)
 	)
-	(global_label "~{MRESET}"
-		(shape input)
+	(global_label "~{BUS_RESET}"
+		(shape output)
 		(at 59.69 330.2 180)
 		(fields_autoplaced yes)
@@
 		)
 		(property "Intersheetrefs" "${INTERSHEET_REFS}"
-			(at 49.5083 330.2 0)
+			(at 46.1821 330.2 0)
 			(hide yes)
 			(show_name no)

Commit message: page 12 done
Parts:
- renumbered R13 to R12
Changed lines of the file:
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@@
 		(in_pos_files yes)
 		(dnp no)
-		(property "Reference" "R13"
+		(property "Reference" "R12"
 			(at 80.01 246.126 90)
 			(show_name no)
@@
 			(project "S8000_CPU"
 				(path "/cee545ba-d57c-4b2c-bcb3-989a68b0ecfa/ab8f6896-63aa-4318-b4ac-54bd1f3ca919"
-					(reference "R13")
+					(reference "R12")
 					(unit 1)
 				)
