File: CircuitDiagrams/S8000_CPU/S8000_CPU_08.kicad_sch (KiCad schematic)
At the start: 16 parts, among them U14 74113, U15 74113, U17 7400, U20 74113, U21 7432, U30 7410, U32 7404, U35 7407, U5 7408, U6 7402, U86 Z8010, U87 Z8010, U88 Z8010

Commit message: Footprints
Parts:
- U14, U15, U17, U20, U21, U30, U32, U35, U5, U6: footprint (none) -> Package_DIP:DIP-14_W7.62mm
- U86, U87, U88: footprint (none) -> Package_DIP:DIP-48_W15.24mm
Changed lines of the file:
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@@
 			)
 		)
-		(property "Footprint" ""
+		(property "Footprint" "Package_DIP:DIP-48_W15.24mm"
 			(at 374.65 440.69 0)
 			(hide yes)
@@
 			)
 		)
-		(property "Footprint" ""
+		(property "Footprint" "Package_DIP:DIP-14_W7.62mm"
 			(at 107.95 303.53 0)
 			(hide yes)
@@
 			)
 		)
-		(property "Footprint" ""
+		(property "Footprint" "Package_DIP:DIP-14_W7.62mm"
 			(at 250.19 299.72 0)
 			(hide yes)
@@
 			)
 		)
-		(property "Footprint" ""
+		(property "Footprint" "Package_DIP:DIP-14_W7.62mm"
 			(at 209.55 312.42 0)
 			(hide yes)
@@
 			)
 		)
-		(property "Footprint" ""
+		(property "Footprint" "Package_DIP:DIP-14_W7.62mm"
 			(at 402.59 307.34 0)
 			(hide yes)
@@
 			)
 		)
-		(property "Footprint" ""
+		(property "Footprint" "Package_DIP:DIP-14_W7.62mm"
 			(at 275.59 302.26 0)
 			(hide yes)
@@
 			)
 		)
-		(property "Footprint" ""
+		(property "Footprint" "Package_DIP:DIP-48_W15.24mm"
 			(at 120.65 440.69 0)
 			(hide yes)
@@
 			)
 		)
-		(property "Footprint" ""
+		(property "Footprint" "Package_DIP:DIP-14_W7.62mm"
 			(at 344.17 307.34 0)
 			(hide yes)
@@
 			)
 		)
-		(property "Footprint" ""
+		(property "Footprint" "Package_DIP:DIP-14_W7.62mm"
 			(at 377.19 304.8 0)
 			(hide yes)
@@
 			)
 		)
-		(property "Footprint" ""
+		(property "Footprint" "Package_DIP:DIP-14_W7.62mm"
 			(at 129.54 330.2 0)
 			(hide yes)
@@
 			)
 		)
-		(property "Footprint" ""
+		(property "Footprint" "Package_DIP:DIP-14_W7.62mm"
 			(at 88.9 285.75 0)
 			(hide yes)
@@
 			)
 		)
-		(property "Footprint" ""
+		(property "Footprint" "Package_DIP:DIP-48_W15.24mm"
 			(at 247.65 440.69 0)
 			(hide yes)
@@
 			)
 		)
-		(property "Footprint" ""
+		(property "Footprint" "Package_DIP:DIP-14_W7.62mm"
 			(at 173.99 314.96 0)
 			(hide yes)
@@
 			)
 		)
-		(property "Footprint" ""
+		(property "Footprint" "Package_DIP:DIP-14_W7.62mm"
 			(at 344.17 323.85 0)
 			(hide yes)

Commit message: Page 10
Parts:
- renumbered U15 to U20
Changed lines of the file:
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@@
 		(in_pos_files yes)
 		(dnp no)
-		(property "Reference" "U15"
+		(property "Reference" "U20"
 			(at 250.19 292.1 0)
 			(show_name no)
@@
 			(project "S8000_CPU"
 				(path "/cee545ba-d57c-4b2c-bcb3-989a68b0ecfa/200ddfb8-e065-44f3-b509-f21dbfc08653"
-					(reference "U15")
+					(reference "U20")
 					(unit 2)
 				)

Commit message: page 12 done
Parts:
- renumbered U6 to U18, U5 to U3
Changed lines of the file:
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@@
 		(in_pos_files yes)
 		(dnp no)
-		(property "Reference" "U5"
+		(property "Reference" "U3"
 			(at 209.55 303.784 0)
 			(show_name no)
@@
 			(project "S8000_CPU"
 				(path "/cee545ba-d57c-4b2c-bcb3-989a68b0ecfa/200ddfb8-e065-44f3-b509-f21dbfc08653"
-					(reference "U5")
+					(reference "U3")
 					(unit 4)
 				)
@@
 		(in_pos_files yes)
 		(dnp no)
-		(property "Reference" "U6"
+		(property "Reference" "U18"
 			(at 344.17 298.196 0)
 			(show_name no)
@@
 			(project "S8000_CPU"
 				(path "/cee545ba-d57c-4b2c-bcb3-989a68b0ecfa/200ddfb8-e065-44f3-b509-f21dbfc08653"
-					(reference "U6")
+					(reference "U18")
 					(unit 4)
 				)
