File: CircuitDiagrams/S8000_CPU/S8000_CPU_10.kicad_sch (KiCad schematic)
At the start: 37 parts, among them U1 7404, U12 74244, U15 7402, U16 7451, U17 7400, U18 7402, U2 7410, U21 7432, U22 7432, U23 7410, U29 7404, U3 7408, U30 7410, U34 74260, U38 7408, U52 7485, U53 7485, U55 74138, U61 74260, U7 7474, U71 74373, U72 74373, U73 74244

Commit message: page 11 done
Connections:
- net IN/~{S}: now also E12., E2., U17.10, U2.10
- net NONSEGUSER: now also E5., U2.9
- net ~{SEGVIOL}: now also E9., R1.2; no longer E7., U17.3
- net NONSEG1_DEF: no longer names the net of E11., U17.2, U3.1, U7.8 (~{Q}), U72.1 (OE)
- net NONSEG2_DEF: no longer names the net of E3., E4., U15.5, U17.8, U30.5
- net NONSEG2_DEF: no longer E2., E5., U2.10, U2.9
- new net: E7., U17.3
Other:
- note removed: "NONSEG3_DEF"
Changed lines of the file:
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@@
 		)
 	)
-	(text "NONSEG3_DEF"
-		(exclude_from_sim no)
-		(at 414.528 371.094 0)
-		(effects
-			(font
-				(size 1.27 1.27)
-				(color 0 0 0 1)
-			)
-		)
-	)
 	(text "(Sh. 3)"
 		(exclude_from_sim no)
@@
 		)
 	)
-	(text "NONSEG3_DEF"
-		(exclude_from_sim no)
-		(at 377.698 371.094 0)
-		(effects
-			(font
-				(size 1.27 1.27)
-				(color 0 0 0 1)
-			)
-		)
-	)
 	(text "1.1"
 		(exclude_from_sim no)
@@
 		)
 	)
+	(polyline
+		(pts
+			(xy 391.7562 323.8527) (xy 400.6908 323.8527)
+		)
+		(stroke
+			(width 0)
+			(type default)
+		)
+	)
 	(wire
 		(pts
@@
 		)
 	)
+	(polyline
+		(pts
+			(xy 400.7465 341.6327) (xy 400.7465 336.7302)
+		)
+		(stroke
+			(width 0)
+			(type default)
+		)
+	)
 	(wire
 		(pts
@@
 		)
 	)
+	(polyline
+		(pts
+			(xy 391.873 374.6299) (xy 400.8076 374.6299)
+		)
+		(stroke
+			(width 0)
+			(type default)
+		)
+	)
 	(wire
 		(pts
@@
 		)
 	)
+	(polyline
+		(pts
+			(xy 400.6491 297.18) (xy 400.6491 292.2775)
+		)
+		(stroke
+			(width 0)
+			(type default)
+		)
+	)
 	(wire
 		(pts
@@
 		)
 	)
+	(polyline
+		(pts
+			(xy 400.8076 374.6299) (xy 400.8076 369.7274)
+		)
+		(stroke
+			(width 0)
+			(type default)
+		)
+	)
 	(wire
 		(pts
@@
 		)
 	)
+	(polyline
+		(pts
+			(xy 391.8119 341.6327) (xy 400.7465 341.6327)
+		)
+		(stroke
+			(width 0)
+			(type default)
+		)
+	)
 	(wire
 		(pts
@@
 		)
 	)
+	(polyline
+		(pts
+			(xy 400.6908 323.8527) (xy 400.6908 318.9502)
+		)
+		(stroke
+			(width 0)
+			(type default)
+		)
+	)
 	(wire
 		(pts
@@
 		)
 	)
+	(polyline
+		(pts
+			(xy 391.7145 297.18) (xy 400.6491 297.18)
+		)
+		(stroke
+			(width 0)
+			(type default)
+		)
+	)
 	(wire
 		(pts
@@
 		)
 	)
-	(label "NONSEG2_DEF"
-		(at 408.94 318.77 0)
-		(effects
-			(font
-				(size 1.27 1.27)
-			)
-			(justify left top)
-		)
-	)
 	(label "BRK1"
 		(at 303.53 251.46 180)
@@
 		)
 	)
-	(label "NONSEG1_DEF"
-		(at 407.67 292.1 0)
-		(effects
-			(font
-				(size 1.27 1.27)
-			)
-			(justify left top)
-		)
-	)
 	(label "BRK2"
 		(at 349.25 238.76 0)
@@
 		)
 	)
-	(label "NONSEG2_DEF"
-		(at 383.54 318.77 180)
-		(effects
-			(font
-				(size 1.27 1.27)
-			)
-			(justify right top)
-		)
-	)
 	(label "ADIN1"
 		(at 251.46 195.58 0)
@@
 		)
 	)
-	(label "NONSEG2_DEF"
-		(at 408.94 336.55 0)
-		(effects
-			(font
-				(size 1.27 1.27)
-			)
-			(justify left top)
-		)
-	)
 	(label "BRK3"
 		(at 349.25 241.3 0)
@@
 		)
 	)
-	(label "NONSEG1_DEF"
-		(at 383.54 292.1 180)
-		(effects
-			(font
-				(size 1.27 1.27)
-			)
-			(justify right top)
-		)
-	)
 	(label "SN2"
 		(at 76.2 242.57 0)
@@
 		)
 	)
-	(label "NONSEG2_DEF"
-		(at 383.54 336.55 180)
-		(effects
-			(font
-				(size 1.27 1.27)
-			)
-			(justify right top)
-		)
-	)
 	(label "BRK6"
 		(at 303.53 200.66 180)
@@
 		)
 	)
+	(global_label "NONSEGUSER"
+		(shape input)
+		(at 410.21 336.55 270)
+		(fields_autoplaced yes)
+		(effects
+			(font
+				(size 0.01 0.01)
+			)
+			(justify right)
+		)
+		(property "Intersheetrefs" "${INTERSHEET_REFS}"
+			(at 410.21 352.1142 90)
+			(hide yes)
+			(show_name no)
+			(do_not_autoplace no)
+			(effects
+				(font
+					(size 1.27 1.27)
+				)
+				(justify right)
+			)
+		)
+	)
 	(global_label "~{SELSYSBAKREG}"
 		(shape input)
@@
 		)
 	)
+	(global_label "~{SEGVIOL}"
+		(shape output)
+		(at 372.11 383.54 0)
+		(fields_autoplaced yes)
+		(effects
+			(font
+				(size 0.01 0.01)
+			)
+			(justify left)
+		)
+		(property "Intersheetrefs" "${INTERSHEET_REFS}"
+			(at 372.1947 383.54 0)
+			(hide yes)
+			(show_name no)
+			(do_not_autoplace no)
+			(effects
+				(font
+					(size 1.27 1.27)
+				)
+				(justify left)
+			)
+		)
+	)
 	(global_label "POWERFAIL"
 		(shape input)
@@
 		)
 	)
+	(global_label "IN{slash}~{S}"
+		(shape input)
+		(at 414.02 318.77 270)
+		(fields_autoplaced yes)
+		(effects
+			(font
+				(size 0.01 0.01)
+			)
+			(justify right)
+		)
+		(property "Intersheetrefs" "${INTERSHEET_REFS}"
+			(at 414.02 326.2305 90)
+			(hide yes)
+			(show_name no)
+			(do_not_autoplace no)
+			(effects
+				(font
+					(size 1.27 1.27)
+				)
+				(justify right)
+			)
+		)
+	)
 	(global_label "ISNAD0"
 		(shape input)
@@
 		)
 	)
-	(global_label "~{SEGVIOL}"
-		(shape output)
-		(at 359.41 369.57 0)
+	(global_label "IN{slash}~{S}"
+		(shape input)
+		(at 414.02 292.1 270)
 		(fields_autoplaced yes)
 		(effects
 			(font
-				(size 1.27 1.27)
+				(size 0.01 0.01)
 			)
-			(justify left)
+			(justify right)
 		)
 		(property "Intersheetrefs" "${INTERSHEET_REFS}"
-			(at 370.0757 369.57 0)
+			(at 414.02 299.5605 90)
 			(hide yes)
 			(show_name no)
@@
 					(size 1.27 1.27)
 				)
-				(justify left)
+				(justify right)
 			)
 		)

Commit message: page 12 done
Parts:
- renumbered U7 to U5
Changed lines of the file:
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@@
 		(in_pos_files yes)
 		(dnp no)
-		(property "Reference" "U7"
+		(property "Reference" "U5"
 			(at 169.418 221.488 0)
 			(show_name no)
@@
 			(project "S8000_CPU"
 				(path "/cee545ba-d57c-4b2c-bcb3-989a68b0ecfa/4e879ea0-dc92-483b-ab60-ba7ce561d4ea"
-					(reference "U7")
+					(reference "U5")
 					(unit 2)
 				)
