File: CircuitDiagrams/S8000_CPU/S8000_CPU_12.kicad_sch (KiCad schematic)
At the start: 0 parts

Commit message: page 12 done
Parts:
- added R13: 1k, Resistor_THT:R_Axial_DIN0207_L6.3mm_D2.5mm_P7.62mm_Horizontal, symbol Device:R_US
- added U11: 74240, Package_DIP:DIP-20_W7.62mm, symbol 74xx:74LS240_Split
- added U2: 7410, symbol 74xx:74LS10
- added U24, U39: 74138, symbol 74xx:74LS138
- added U29, U32: 7404, symbol 74xx:74LS04
- added U40: 7474, symbol 74xx:74LS74
- added U41: 7432, symbol 74xx:74LS32
- added U42: 7408, symbol 74xx:74LS08
- added U45: 74133, symbol 74xx:74LS133
- added U6: 7400, symbol 74xx:74LS00
- added U61: 74260, symbol S8000:74LS260
- added U7: 7420, symbol 74xx:74LS20
Connections:
- new net: U24.4 (E1), U39.4 (E1), U45.9, U61.1, U7.4
- new net: U39.5 (E2), U40.8 (~{Q}), U41.9, U61.12
- new net: U11.3, U39.6 (E3), U6.10, U61.2
- new net: U6.1, U61.5
- new net: U40.1 (~{R}), U40.9 (Q)
- new net: U42.10, U42.12, U6.3
- new net: U2.12, U42.13
- new net: U41.6, U7.1
- new net: U2.13, U40.5 (Q), U6.9
- new net: U41.8, U42.9
- new net: R13.2, U45.10, U45.11
- new net: U41.11, U42.2
- new net: U42.1, U6.8
- new net: U29.8, U40.2 (D), U45.12
- new net +5V: R13.1, U24.16 (VCC), U39.16 (VCC), U40.13 (~{R}), U40.4 (~{S})
- new net CTC 0 ~{CE}: U39.11 (O4)
- new net CTC 1 ~{CE}: U39.10 (O5)
- new net CTC 2 ~{CE}: U39.9 (O6)
- new net GND: U24.8 (GND), U39.8 (GND), U40.12 (D)
- new net IMEML: U7.5
- new net INT PHI: U40.3 (C)
- new net IR/~{W}: U2.2
- new net LAD0: U45.14
- new net LAD10: U45.1
- new net LAD11: U45.4
- new net LAD12: U45.5
- new net LAD13: U45.6
- new net LAD14: U45.7
- new net LAD15: U45.15
- new net LAD3: U24.1 (A0), U39.1 (A0), U61.3
- new net LAD4: U24.2 (A1), U39.2 (A1), U61.13
- new net LAD5: U24.3 (A2), U39.3 (A2), U6.2
- new net LAD6: U11.17, U24.6 (E3)
- new net LAD7: U45.13
- new net LAD8: U45.3
- new net LAD9: U45.2
- new net NON BD: U32.6
- new net PIO ~{CE}: U39.7 (O7)
- new net SIO 0 ~{CE}: U39.15 (O0)
- new net SIO 1 ~{CE}: U39.14 (O1)
- new net SIO 2 ~{CE}: U39.13 (O2)
- new net SIO 3 ~{CE}: U39.12 (O3)
- new net SYS IEO 2: U41.4
- new net ~{IAS}: U40.10 (~{S})
- new net ~{IDS}: U24.5 (E2), U40.11 (C), U41.12
- new net ~{IF1LOBYTE}: U24.9 (O6)
- new net ~{IRQ}: U42.3
- new net ~{I/O REF}: U29.9
- new net ~{M1}: U42.8
- new net ~{NON BD}: U32.5, U7.6
- new net ~{ONBDNMI}: U7.2
- new net ~{RD}: U42.11
- new net ~{SELNBRKREG}: U24.13 (O2)
- new net ~{SELSNVIOLREG}: U24.12 (O3)
- new net ~{SELSYSBAKREG}: U24.14 (O1)
- new net ~{SOFTRESET}: U24.7 (O7)
- new net ~{SYS CONFIG}: U24.15 (O0)
- new net ~{TRPLOBYTE}: U24.10 (O5)
- new net ~{VIACK}: U2.1, U41.10, U41.13, U41.5
- no-connect marks 0 -> 2
Other:
- note added: "(Sh. 10)"
- note added: "(Sh. 11)"
- note added: "(Sh. 13)"
- note added: "(Sh. 13,14)"
- note added: "(Sh. 14)"
- note added: "(Sh. 2)"
- note added: "(Sh. 3)"
- note added: "(Sh. 4)"
- note added: "(Sh. 4,5,6,7)"
- note added: "(Sh. 5)"
- note added: "(Sh. 6)"
- note added: "(Sh. 7)"
- note added: "1.1"
- note added: "FF81"
- note added: "FF89"
- note added: "FF91"
- note added: "FF99"
- note added: "FFA1"
- note added: "FFA9"
- note added: "FFB1"
- note added: "FFB9"
- note added: "FFC1"
- note added: "FFC9"
- note added: "FFD1"
- note added: "FFD9"
- note added: "FFE9"
- note added: "FFF1"
- note added: "FFF9"
- note added: "Oliver Lehmann <lehmann@ans-netz.de>"
- note added: "Peripheral Handshaking Logic (U24, U39)"
- note added: "Zilog S8000 CPU"

Commit message: U98 is a 74S161/93S16
Changed lines of the file:
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@@
 	(text "(Sh. 2)"
 		(exclude_from_sim no)
-		(at 39.37 25.4 0)
+		(at 39.37 21.59 0)
 		(effects
 			(font
@@
 	)
 	(junction
-		(at 179.07 78.74)
+		(at 142.24 78.74)
 		(diameter 0)
 		(color 0 0 0 0)
@@
 	)
 	(junction
-		(at 88.9 25.4)
+		(at 88.9 21.59)
 		(diameter 0)
 		(color 0 0 0 0)
@@
 	(bus
 		(pts
-			(xy 165.1 25.4) (xy 88.9 25.4)
+			(xy 165.1 21.59) (xy 88.9 21.59)
 		)
 		(stroke
@@
 	(bus
 		(pts
-			(xy 88.9 25.4) (xy 88.9 120.65)
+			(xy 88.9 21.59) (xy 88.9 120.65)
 		)
 		(stroke
@@
 	(wire
 		(pts
-			(xy 179.07 78.74) (xy 142.24 78.74)
-		)
-		(stroke
-			(width 0)
-			(type default)
-		)
-	)
-	(wire
-		(pts
 			(xy 125.73 226.06) (xy 125.73 223.52)
 		)
@@
 	(bus
 		(pts
-			(xy 165.1 68.58) (xy 165.1 25.4)
+			(xy 165.1 68.58) (xy 165.1 21.59)
 		)
 		(stroke
@@
 	(wire
 		(pts
-			(xy 179.07 78.74) (xy 184.15 78.74)
-		)
-		(stroke
-			(width 0)
-			(type default)
-		)
-	)
-	(wire
-		(pts
-			(xy 179.07 25.4) (xy 184.15 25.4)
+			(xy 142.24 25.4) (xy 184.15 25.4)
 		)
 		(stroke
@@
 		)
 	)
+	(wire
+		(pts
+			(xy 142.24 78.74) (xy 184.15 78.74)
+		)
+		(stroke
+			(width 0)
+			(type default)
+		)
+	)
 	(bus
 		(pts
-			(xy 88.9 25.4) (xy 59.69 25.4)
+			(xy 88.9 21.59) (xy 59.69 21.59)
 		)
 		(stroke
@@
 	(wire
 		(pts
-			(xy 179.07 78.74) (xy 179.07 25.4)
+			(xy 142.24 78.74) (xy 142.24 25.4)
 		)
 		(stroke
@@
 	(global_label "LAD[0..15]"
 		(shape input)
-		(at 59.69 25.4 180)
+		(at 59.69 21.59 180)
 		(fields_autoplaced yes)
 		(effects
@@
 		)
 		(property "Intersheetrefs" "${INTERSHEET_REFS}"
-			(at 46.7866 25.4 0)
-			(hide yes)
-			(show_name no)
+			(at 46.7866 21.59 0)
+			(hide yes)
+			(show_name no)
