File: CircuitDiagrams/S8000_CPU/S8000_CPU_13.kicad_sch (KiCad schematic)
At the start: 0 parts

Commit message: add notes
Other:
- note added: "1.1"
- note added: "Address/Data Buffers and Steering Logic Byte Swap Buffer (U112)"
- note added: "Oliver Lehmann <lehmann@ans-netz.de>"
- note added: "Zilog S8000 CPU"
Changed lines of the file:
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@@
 	(generator "eeschema")
 	(generator_version "10.0")
-	(paper "A4")
+	(paper "A2")
+	(text "Zilog S8000 CPU"
+		(exclude_from_sim no)
+		(at 497.586 399.796 0)
+		(effects
+			(font
+				(size 2.032 2.032)
+				(thickness 0.4064)
+				(bold yes)
+			)
+		)
+	)
+	(text "1.1"
+		(exclude_from_sim no)
+		(at 572.262 404.368 0)
+		(effects
+			(font
+				(size 1.524 1.524)
+			)
+			(justify left bottom)
+		)
+	)
+	(text "Address/Data Buffers and Steering Logic\nByte Swap Buffer (U112)"
+		(exclude_from_sim no)
+		(at 474.726 390.652 0)
+		(effects
+			(font
+				(size 1.778 1.778)
+			)
+			(justify left bottom)
+		)
+	)
+	(text "Oliver Lehmann <lehmann@ans-netz.de>"
+		(exclude_from_sim no)
+		(at 500.38 407.67 0)
+		(effects
+			(font
+				(size 1.778 1.778)
+			)
+			(justify left bottom)
+		)
+	)
 )
